File: springreverb_lm386.kicad_sch (KiCad schematic)
At the start: 67 parts, among them J1 IN, J10 VR2_3, J11 VR_2_2, J12 VR_2GND, J13 To, J14 FromSW, J15 To_Tank, J16 From_Tank, J17 FromGND, J18 From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

Commit message: フィルムコンデンサを変更
Parts:
- C14, C2: footprint Capacitor_THT:C_Rect_L10.3mm_W5.0mm_P7.50mm_MKS4 -> MyLibrary:9.3_4.3_p7.5
- C6: footprint MyLibrary:10.5_5.0_p7.5 -> MyLibrary:9.3_4.3_p7.5
- C7: footprint MyLibrary:10.5_5.0_p7.5 -> MyLibrary:11.2_4.3_p10
- H1, H2, H3, H4: footprint MountingHole:MountingHole_3.2mm_M3 -> MyLibrary:MountingHole_3.2mm_M3
Changed lines of the file:
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@@
 			)
 		)
-		(property "Footprint" "MyLibrary:10.5_5.0_p7.5"
+		(property "Footprint" "MyLibrary:9.3_4.3_p7.5"
 			(at 97.79 138.43 0)
 			(hide yes)
@@
 			)
 		)
-		(property "Footprint" "MountingHole:MountingHole_3.2mm_M3"
+		(property "Footprint" "MyLibrary:MountingHole_3.2mm_M3"
 			(at 21.59 180.34 0)
 			(hide yes)
@@
 			)
 		)
-		(property "Footprint" "Capacitor_THT:C_Rect_L10.3mm_W5.0mm_P7.50mm_MKS4"
+		(property "Footprint" "MyLibrary:9.3_4.3_p7.5"
 			(at 134.62 146.05 0)
 			(hide yes)
@@
 			)
 		)
-		(property "Footprint" "MountingHole:MountingHole_3.2mm_M3"
+		(property "Footprint" "MyLibrary:MountingHole_3.2mm_M3"
 			(at 46.99 181.61 0)
 			(hide yes)
@@
 			)
 		)
-		(property "Footprint" "MountingHole:MountingHole_3.2mm_M3"
+		(property "Footprint" "MyLibrary:MountingHole_3.2mm_M3"
 			(at 68.58 181.61 0)
 			(hide yes)
@@
 			)
 		)
-		(property "Footprint" "MyLibrary:10.5_5.0_p7.5"
+		(property "Footprint" "MyLibrary:11.2_4.3_p10"
 			(at 97.79 147.32 0)
 			(hide yes)
@@
 			)
 		)
-		(property "Footprint" "MountingHole:MountingHole_3.2mm_M3"
+		(property "Footprint" "MyLibrary:MountingHole_3.2mm_M3"
 			(at 87.63 181.61 0)
 			(hide yes)
@@
 			)
 		)
-		(property "Footprint" "Capacitor_THT:C_Rect_L10.3mm_W5.0mm_P7.50mm_MKS4"
+		(property "Footprint" "MyLibrary:9.3_4.3_p7.5"
 			(at 38.1 130.81 0)
 			(hide yes)
